Commit message: Refactor arm movement logic and update URDF model handling

File: src/cyberwave_hackaton/manipulation/models/piper_description.urdf (robot description, URDF)
Before this commit: robot piper, 11 links, 10 joints
Links:
- removed link link7
- removed link link8
Joints:
- removed joint joint7
- removed joint joint8
